File: hardware/kicad/NOP100.kicad_pcb (KiCad board)
At the start: 2 copper layers, 100 x 85 mm, 74 parts, among them J2 CAN, Q1 BSS138, Q2 BSS138, SW1 PRG, SW2 INSTANCE, SW3 BUS, U1 MCP2551-I-P, U101 74HC165, U2 TMR-2-2411, U3 74HCT595, U4 74HCT595, U5 Teensy_4.0

Commit message: Add testpomts
Connections:
- net D16 renamed /D16
- net D17 renamed /D17
- net D18 renamed /D18
- net D19 renamed /D19
- net D20 renamed /D20
- net D21 renamed /D21
- net D22 renamed /D22
- net D23 renamed /D23
- net D5 renamed /D5
- net D6 renamed /D6
- net D7 renamed /D7
- net D8 renamed /D8
- net D9 renamed /D9
Other:
- board text removed: "NMEA 2000 Temperature Sensor Module"
- board text removed: "PWR/TX"
- board text removed: "TSENSE"

Commit message: Documentation
Parts:
- renumbered C5 to C1001, C1 to C1002, C3 to C1003, C101 to C1004, C4 to C1005, C2 to C1006, D5 to D1001, D1 to D1002, D2 to D1003, D3 to D1004, D4 to D1005, D18 to D1006, D19 to D1007, D20 to D1008, D21 to D1009, D6 to D1010, D7 to D1011, D8 to D1012, D9 to D1013, D22 to D1014, D23 to D1015, D24 to D1016, D25 to D1017, F1 to F1001, J2 to J1001, Q1 to Q1001, Q2 to Q1002, R4 to R1001, R5 to R1002, R6 to R1003, R7 to R1004, R3 to R1005, R1 to R1006, R2 to R1007, R101 to R1008, R102 to R1009, R103 to R1010, R104 to R1011, R105 to R1012, R106 to R1013, R107 to R1014, R108 to R1015, R28 to R1016, R29 to R1017, R30 to R1018, R31 to R1019, R32 to R1020, R33 to R1021, R34 to R1022, R35 to R1023, R40 to R1024, R41 to R1025, R42 to R1026, R43 to R1027, R44 to R1028, R45 to R1029, R46 to R1030, R47 to R1031, SW3 to SW1001, SW2 to SW1002, SW1 to SW1003, U2 to U1001, U1 to U1002, U5 to U1003, U101 to U1004, U4 to U1005, U3 to U1006

Commit message: Silkscreen
Parts:
- SW1002: value INSTANCE -> ADDR/VALUE
