File: hardware/kicad/NOP100.kicad_sch (KiCad schematic)
At the start: 45 parts, among them CON1 CLICK MODULE 0, CON2 CLICK MODULE 1, J1 CAN, Q1 BSS138, Q2 BSS138, SW1 BUS, SW2 SW_Push, U1 MURATA_MEJ2*, U2 MCP2551-I-P, U3 Teensy_4.0, U4 74HC165, U6 NCS1S1203SC

Commit message: Tweaks
Connections:
- net +3V3: now also R10.2, R11.2, R12.2, R13.2, R14.2, R15.2, R16.2, R9.2; no longer HI1.1 (CM), LO1.1 (CM)
- net GND: now also HI1.1 (CM), LO1.1 (CM); no longer R10.2, R11.2, R12.2, R13.2, R14.2, R15.2, R16.2, R9.2
Other:
- note added: "MIKROBUS"
- note removed: "MIKROBUS INTERFACE"
- moved on the sheet: C4, D2, R10, R11, R12, R13, R14, R15, R16, R17, R8, R9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

Commit message: Tweaks
Parts:
- added J10, J2, J3, J4, J5, J6, J8, J9: Conn_01x03, pdjr:RS_8971054, symbol Connector_Generic:Conn_01x03
- added J7: Conn_02x05_Odd_Even, Connector_PinSocket_2.54mm:PinSocket_2x05_P2.54mm_Vertical, symbol Connector_Generic:Conn_02x05_Odd_Even
Connections:
- new net OW0: J3.3 (Pin_3), J7.9 (Pin_9)
- new net OW1: J6.3 (Pin_3), J7.10 (Pin_10)
- new net OW2: J2.3 (Pin_3), J7.7 (Pin_7)
- new net OW3: J7.8 (Pin_8), J8.3 (Pin_3)
- new net OW4: J4.3 (Pin_3), J7.5 (Pin_5)
- new net OW5: J7.6 (Pin_6), J9.3 (Pin_3)
- new net OW6: J5.3 (Pin_3), J7.3 (Pin_3)
- new net OW7: J10.3 (Pin_3), J7.4 (Pin_4)
- new net OW_GND: J10.1 (Pin_1), J2.1 (Pin_1), J3.1 (Pin_1), J4.1 (Pin_1), J5.1 (Pin_1), J6.1 (Pin_1), J7.2 (Pin_2), J8.1 (Pin_1), J9.1 (Pin_1)
- new net OW_VCC: J10.2 (Pin_2), J2.2 (Pin_2), J3.2 (Pin_2), J4.2 (Pin_2), J5.2 (Pin_2), J6.2 (Pin_2), J7.1 (Pin_1), J8.2 (Pin_2), J9.2 (Pin_2)
Other:
- note added: "1-WIRE BUS"
- moved on the sheet: C3, CON1, CON2, JP1, R18, R19, R20, R21, U3
